Commit message: fixed URDF model, added launch for Gazebo

File: ros2_ws/src/padwq_description/urdf/padwq_original.urdf.xacro (robot description, xacro)
@@ -1,4 +1,4 @@
 <?xml version="1.0"?>
-<robot name="padwq">
+<robot name="padwq_robot">
     <material name="silver">
         <color rgba="0.700 0.700 0.700 1.000"/>
@@ -76,5 +76,5 @@
             <origin rpy="-1.57 0.47 1.57" xyz="-0.07 -0.147 0.074"/>
             <geometry>
-                <mesh filename="file://$(find padwq)/leg1_5.stl" scale="-0.001 0.001 0.001"/>
+                <mesh filename="file://$(find padwq_description)/meshes/leg1_5.stl" scale="-0.001 0.001 0.001"/>
             </geometry>
             <material name="silver"/>
@@ -91,5 +91,5 @@
             <origin rpy="-1.57 -0.47 -1.57" xyz="0.063 0.0492 0.1717"/>
             <geometry>
-                <mesh filename="file://$(find padwq)/leg4.stl" scale="0.001 0.001 0.001"/>
+                <mesh filename="file://$(find padwq_description)/meshes/leg4.stl" scale="0.001 0.001 0.001"/>
             </geometry>
             <material name="silver"/>
@@ -105,5 +105,5 @@
             <origin rpy="0 -1.57 1.57" xyz="0 0 -0.0269"/>
             <geometry>
-                <mesh filename="file://$(find padwq)/ball_leg4_1.stl" scale="0.001 0.001 0.001"/>
+                <mesh filename="file://$(find padwq_description)/meshes/ball_leg4_1.stl" scale="0.001 0.001 0.001"/>
             </geometry>
             <material name="silver"/>
@@ -137,5 +137,5 @@
             <origin rpy="-1.57 0.47 1.57" xyz="-0.07 -0.147 0.074"/>
             <geometry>
-                <mesh filename="file://$(find padwq)/leg1_5.stl" scale="-0.001 0.001 0.001"/>
+                <mesh filename="file://$(find padwq_description)/meshes/leg1_5.stl" scale="-0.001 0.001 0.001"/>
             </geometry>
             <material name="silver"/>
@@ -152,5 +152,5 @@
             <origin rpy="-1.57 -0.47 -1.57" xyz="0.063 0.0492 0.1717"/>
             <geometry>
-                <mesh filename="file://$(find padwq)/leg4.stl" scale="0.001 0.001 0.001"/>
+                <mesh filename="file://$(find padwq_description)/meshes/leg4.stl" scale="0.001 0.001 0.001"/>
             </geometry>
             <material name="silver"/>
@@ -166,5 +166,5 @@
             <origin rpy="0 -1.57 1.57" xyz="0 0 -0.0269"/>
             <geometry>
-                <mesh filename="file://$(find padwq)/ball_leg4_1.stl" scale="0.001 0.001 0.001"/>
+                <mesh filename="file://$(find padwq_description)/meshes/ball_leg4_1.stl" scale="0.001 0.001 0.001"/>
             </geometry>
             <material name="silver"/>
@@ -198,5 +198,5 @@
             <origin rpy="-1.57 -0.47 -1.57" xyz="0.07 -0.147 0.074"/>
             <geometry>
-                <mesh filename="file://$(find padwq)/leg1_5.stl" scale="0.001 0.001 0.001"/>
+                <mesh filename="file://$(find padwq_description)/meshes/leg1_5.stl" scale="0.001 0.001 0.001"/>
             </geometry>
             <material name="silver"/>
@@ -213,5 +213,5 @@
             <origin rpy="-1.57 -0.47 -1.57" xyz="0.063 0.0492 0.1717"/>
             <geometry>
-                <mesh filename="file://$(find padwq)/leg4.stl" scale="0.001 0.001 0.001"/>
+                <mesh filename="file://$(find padwq_description)/meshes/leg4.stl" scale="0.001 0.001 0.001"/>
             </geometry>
             <material name="silver"/>
@@ -227,5 +227,5 @@
             <origin rpy="0 -1.57 1.57" xyz="0 0 -0.0269"/>
             <geometry>
-                <mesh filename="file://$(find padwq)/ball_leg4_1.stl" scale="0.001 0.001 0.001"/>
+                <mesh filename="file://$(find padwq_description)/meshes/ball_leg4_1.stl" scale="0.001 0.001 0.001"/>
             </geometry>
             <material name="silver"/>
@@ -259,5 +259,5 @@
             <origin rpy="-1.57 -0.47 -1.57" xyz="0.07 -0.147 0.074"/>
             <geometry>
-                <mesh filename="file://$(find padwq)/leg1_5.stl" scale="0.001 0.001 0.001"/>
+                <mesh filename="file://$(find padwq_description)/meshes/leg1_5.stl" scale="0.001 0.001 0.001"/>
             </geometry>
             <material name="silver"/>
@@ -274,5 +274,5 @@
             <origin rpy="-1.57 -0.47 -1.57" xyz="0.063 0.0492 0.1717"/>
             <geometry>
-                <mesh filename="file://$(find padwq)/leg4.stl" scale="0.001 0.001 0.001"/>
+                <mesh filename="file://$(find padwq_description)/meshes/leg4.stl" scale="0.001 0.001 0.001"/>
             </geometry>
             <material name="silver"/>
@@ -288,5 +288,5 @@
             <origin rpy="0 -1.57 1.57" xyz="0 0 -0.0269"/>
             <geometry>
-                <mesh filename="file://$(find padwq)/ball_leg4_1.stl" scale="0.001 0.001 0.001"/>
+                <mesh filename="file://$(find padwq_description)/meshes/ball_leg4_1.stl" scale="0.001 0.001 0.001"/>
             </geometry>
             <material name="silver"/>
