Commit message: updated controllers

File: ros2_ws/src/padwq_description/urdf/gazebo.xacro (robot description, xacro)
@@ -2,4 +2,17 @@
 <robot xmlns:xacro="http://www.ros.org/wiki/xacro">
     <xacro:macro name="gazebo" params="prefix">
+        <xacro:macro name="foot_surface">
+            <contact>
+                <min_depth>0.001</min_depth>
+            </contact>
+            <mu1>100.0</mu1>
+            <mu2>100.0</mu2>
+            <kp>1e13</kp>
+            <kd>1.0</kd>
+            <minDepth>0.001</minDepth>
+            <bounce_threshold>10000000</bounce_threshold>
+            <maxVel>0.1</maxVel>
+            <fdir1>0 0 0</fdir1>
+        </xacro:macro>
         <gazebo reference="${prefix}base_link">
             <material>Gazebo/White</material>
@@ -28,4 +41,5 @@
         <gazebo reference="${prefix}fl_foot">
             <material>Gazebo/Black</material>
+            <xacro:foot_surface/>
         </gazebo>
         <gazebo reference="${prefix}fr_hip_roll_actuator">
@@ -52,4 +66,5 @@
         <gazebo reference="${prefix}fr_foot">
             <material>Gazebo/Black</material>
+            <xacro:foot_surface/>
         </gazebo>
         <gazebo reference="${prefix}rl_hip_roll_actuator">
@@ -76,4 +91,5 @@
         <gazebo reference="${prefix}rl_foot">
             <material>Gazebo/Black</material>
+            <xacro:foot_surface/>
         </gazebo>
         <gazebo reference="${prefix}rr_hip_roll_actuator">
@@ -100,4 +116,5 @@
         <gazebo reference="${prefix}rr_foot">
             <material>Gazebo/Black</material>
+            <xacro:foot_surface/>
         </gazebo>
     </xacro:macro>

File: ros2_ws/src/padwq_description/urdf/padwq.ros2_control.xacro (robot description, xacro)
@@ -8,66 +8,102 @@
             <joint name="${prefix}fl_hip_roll">
                 <command_interface name="position"/>
-                <state_interface name="position"/>
+                <state_interface name="position">
+                    <param name="initial_value">0.0</param>
+                </state_interface>
                 <state_interface name="velocity"/>
+                <state_interface name="effort"/>
             </joint>
             <joint name="${prefix}fl_hip_pitch">
                 <command_interface name="position"/>
-                <state_interface name="position"/>
+                <state_interface name="position">
+                    <param name="initial_value">0.0</param>
+                </state_interface>
                 <state_interface name="velocity"/>
+                <state_interface name="effort"/>
             </joint>
             <joint name="${prefix}fl_knee_pitch">
                 <command_interface name="position"/>
-                <state_interface name="position"/>
+                <state_interface name="position">
+                    <param name="initial_value">0.0</param>
+                </state_interface>
                 <state_interface name="velocity"/>
+                <state_interface name="effort"/>
             </joint>
             <joint name="${prefix}fr_hip_roll">
                 <command_interface name="position"/>
-                <state_interface name="position"/>
+                <state_interface name="position">
+                    <param name="initial_value">0.0</param>
+                </state_interface>
                 <state_interface name="velocity"/>
+                <state_interface name="effort"/>
             </joint>
             <joint name="${prefix}fr_hip_pitch">
                 <command_interface name="position"/>
-                <state_interface name="position"/>
+                <state_interface name="position">
+                    <param name="initial_value">0.0</param>
+                </state_interface>
                 <state_interface name="velocity"/>
+                <state_interface name="effort"/>
             </joint>
             <joint name="${prefix}fr_knee_pitch">
                 <command_interface name="position"/>
-                <state_interface name="position"/>
+                <state_interface name="position">
+                    <param name="initial_value">0.0</param>
+                </state_interface>
                 <state_interface name="velocity"/>
+                <state_interface name="effort"/>
             </joint>
             <joint name="${prefix}rl_hip_roll">
                 <command_interface name="position"/>
-                <state_interface name="position"/>
+                <state_interface name="position">
+                    <param name="initial_value">0.0</param>
+                </state_interface>
                 <state_interface name="velocity"/>
+                <state_interface name="effort"/>
             </joint>
             <joint name="${prefix}rl_hip_pitch">
                 <command_interface name="position"/>
-                <state_interface name="position"/>
+                <state_interface name="position">
+                    <param name="initial_value">0.0</param>
+                </state_interface>
                 <state_interface name="velocity"/>
+                <state_interface name="effort"/>
             </joint>
             <joint name="${prefix}rl_knee_pitch">
                 <command_interface name="position"/>
-                <state_interface name="position"/>
+                <state_interface name="position">
+                    <param name="initial_value">0.0</param>
+                </state_interface>
                 <state_interface name="velocity"/>
+                <state_interface name="effort"/>
             </joint>
             <joint name="${prefix}rr_hip_roll">
                 <command_interface name="position"/>
-                <state_interface name="position"/>
+                <state_interface name="position">
+                    <param name="initial_value">0.0</param>
+                </state_interface>
                 <state_interface name="velocity"/>
+                <state_interface name="effort"/>
             </joint>
             <joint name="${prefix}rr_hip_pitch">
                 <command_interface name="position"/>
-                <state_interface name="position"/>
+                <state_interface name="position">
+                    <param name="initial_value">0.0</param>
+                </state_interface>
                 <state_interface name="velocity"/>
+                <state_interface name="effort"/>
             </joint>
             <joint name="${prefix}rr_knee_pitch">
                 <command_interface name="position"/>
-                <state_interface name="position"/>
+                <state_interface name="position">
+                    <param name="initial_value">0.0</param>
+                </state_interface>
                 <state_interface name="velocity"/>
+                <state_interface name="effort"/>
             </joint>
         </ros2_control>
         <gazebo>
             <plugin filename="libgazebo_ros2_control.so" name="gazebo_ros2_control">
-                <parameters>$(find padwq_bringup)/config/padwq_controllers.yaml</parameters>
+                <parameters>$(find padwq_description)/config/controllers.yaml</parameters>
             </plugin>
         </gazebo>

File: ros2_ws/src/padwq_description/urdf/padwq.urdf.xacro (robot description, xacro)
@@ -8,11 +8,8 @@
     <!-- import gazebo description -->
     <xacro:include filename="$(find padwq_description)/urdf/gazebo.xacro"/>
-    <!-- import gazebo control -->
-    <xacro:include filename="$(find padwq_description)/urdf/gazebo.control.xacro"/>
     <!-- import ros2_control description -->
-    <!-- <xacro:include filename="$(find padwq_description)/ros2_control/padwq.ros2_control.xacro"/> -->
+    <xacro:include filename="$(find padwq_description)/urdf/padwq.ros2_control.xacro"/>
     <xacro:padwq prefix="$(arg prefix)"/>
     <xacro:gazebo prefix="$(arg prefix)"/>
-    <xacro:gazebo_control prefix="$(arg prefix)"/>
-    <!-- <xacro:padwq_ros2_control name="padwq" prefix="$(arg prefix)"/> -->
+    <xacro:padwq_ros2_control name="padwq" prefix="$(arg prefix)"/>
 </robot>
