Commit message: add damping

File: ros2_ws/src/padwq_description/urdf/padwq.description.xacro (robot description, xacro)
@@ -31,4 +31,5 @@
             <child link="${prefix}fl_hip_roll_actuator"/>
             <origin rpy="0 ${pi/2} 0" xyz="0.1415 0.07 0"/>
+            <dynamics friction="10.0"/>
         </joint>
         <link name="${prefix}fl_hip_roll_actuator">
@@ -56,4 +57,5 @@
             <origin rpy="0 0 0" xyz="0 0 0"/>
             <limit effort="1000.0" lower="${-30 * deg2rad}" upper="${30 * deg2rad}" velocity="0.7"/>
+            <dynamics friction="10.0"/>
         </joint>
         <link name="${prefix}fl_hip_pitch_connector">
@@ -81,4 +83,5 @@
             <origin rpy="${pi/2} 0 0" xyz="0 ${rdm_l/2} 0.068"/>
             <limit effort="1000.0" lower="${-51 * deg2rad}" upper="${93 * deg2rad}" velocity="0.7"/>
+            <dynamics friction="10.0"/>
         </joint>
         <link name="${prefix}fl_hip_pitch_actuator">
@@ -104,4 +107,5 @@
             <child link="${prefix}fl_knee_pitch_connector"/>
             <origin rpy="0 0 0" xyz="0 0 0"/>
+            <dynamics friction="10.0"/>
         </joint>
         <link name="${prefix}fl_knee_pitch_connector">
@@ -127,4 +131,5 @@
             <child link="${prefix}fl_knee_pitch_actuator"/>
             <origin rpy="0 0 0" xyz="0 0 -0.062"/>
+            <dynamics friction="10.0"/>
         </joint>
         <link name="${prefix}fl_knee_pitch_actuator">
@@ -150,4 +155,5 @@
             <child link="${prefix}fl_upper_link"/>
             <origin rpy="0 0 0" xyz="0 0 0"/>
+            <dynamics friction="10.0"/>
         </joint>
         <link name="${prefix}fl_upper_link">
@@ -175,4 +181,5 @@
             <origin rpy="0 0 0" xyz="0.22 0 0"/>
             <limit effort="1000.0" lower="${-134 * deg2rad}" upper="${-7 * deg2rad}" velocity="0.7"/>
+            <dynamics friction="10.0"/>
         </joint>
         <link name="${prefix}fl_under_link">
@@ -199,4 +206,5 @@
             <child link="${prefix}fl_foot"/>
             <origin rpy="0 0 0" xyz="0.22 0 0"/>
+            <dynamics friction="10.0"/>
         </joint>
         <link name="${prefix}fl_foot">
@@ -221,4 +229,5 @@
             <child link="${prefix}fr_hip_roll_actuator"/>
             <origin rpy="0 ${pi/2} 0" xyz="0.1415 -0.07 0"/>
+            <dynamics friction="10.0"/>
         </joint>
         <link name="${prefix}fr_hip_roll_actuator">
@@ -246,4 +255,5 @@
             <origin rpy="0 0 0" xyz="0 0 0"/>
             <limit effort="1000.0" lower="${-30 * deg2rad}" upper="${30 * deg2rad}" velocity="0.7"/>
+            <dynamics friction="10.0"/>
         </joint>
         <link name="${prefix}fr_hip_pitch_connector">
@@ -271,4 +281,5 @@
             <origin rpy="${pi/2} 0 0" xyz="0 -${rdm_l/2} 0.068"/>
             <limit effort="1000.0" lower="${-51 * deg2rad}" upper="${93 * deg2rad}" velocity="0.7"/>
+            <dynamics friction="10.0"/>
         </joint>
         <link name="${prefix}fr_hip_pitch_actuator">
@@ -294,4 +305,5 @@
             <child link="${prefix}fr_knee_pitch_connector"/>
             <origin rpy="0 0 0" xyz="0 0 0"/>
+            <dynamics friction="10.0"/>
         </joint>
         <link name="${prefix}fr_knee_pitch_connector">
@@ -317,4 +329,5 @@
             <child link="${prefix}fr_knee_pitch_actuator"/>
             <origin rpy="0 0 0" xyz="0 0 0.062"/>
+            <dynamics friction="10.0"/>
         </joint>
         <link name="${prefix}fr_knee_pitch_actuator">
@@ -340,4 +353,5 @@
             <child link="${prefix}fr_upper_link"/>
             <origin rpy="0 0 0" xyz="0 0 0"/>
+            <dynamics friction="10.0"/>
         </joint>
         <link name="${prefix}fr_upper_link">
@@ -365,4 +379,5 @@
             <origin rpy="0 0 0" xyz="0.22 0 0"/>
             <limit effort="1000.0" lower="${-134 * deg2rad}" upper="${-7 * deg2rad}" velocity="0.7"/>
+            <dynamics friction="10.0"/>
         </joint>
         <link name="${prefix}fr_under_link">
@@ -389,4 +404,5 @@
             <child link="${prefix}fr_foot"/>
             <origin rpy="0 0 0" xyz="0.22 0 0"/>
+            <dynamics friction="10.0"/>
         </joint>
         <link name="${prefix}fr_foot">
@@ -411,4 +427,5 @@
             <child link="${prefix}rl_hip_roll_actuator"/>
             <origin rpy="0 ${pi/2} 0" xyz="-0.1415 0.07 0"/>
+            <dynamics friction="10.0"/>
         </joint>
         <link name="${prefix}rl_hip_roll_actuator">
@@ -436,4 +453,5 @@
             <origin rpy="0 0 0" xyz="0 0 0"/>
             <limit effort="1000.0" lower="${-30 * deg2rad}" upper="${30 * deg2rad}" velocity="0.7"/>
+            <dynamics friction="10.0"/>
         </joint>
         <link name="${prefix}rl_hip_pitch_connector">
@@ -461,4 +479,5 @@
             <origin rpy="${pi/2} 0 0" xyz="0 ${rdm_l/2} -0.068"/>
             <limit effort="1000.0" lower="${-51 * deg2rad}" upper="${93 * deg2rad}" velocity="0.7"/>
+            <dynamics friction="10.0"/>
         </joint>
         <link name="${prefix}rl_hip_pitch_actuator">
@@ -484,4 +503,5 @@
             <child link="${prefix}rl_knee_pitch_connector"/>
             <origin rpy="0 0 0" xyz="0 0 0"/>
+            <dynamics friction="10.0"/>
         </joint>
         <link name="${prefix}rl_knee_pitch_connector">
@@ -507,4 +527,5 @@
             <child link="${prefix}rl_knee_pitch_actuator"/>
             <origin rpy="0 0 0" xyz="0 0 -0.062"/>
+            <dynamics friction="10.0"/>
         </joint>
         <link name="${prefix}rl_knee_pitch_actuator">
@@ -530,4 +551,5 @@
             <child link="${prefix}rl_upper_link"/>
             <origin rpy="0 0 0" xyz="0 0 0"/>
+            <dynamics friction="10.0"/>
         </joint>
         <link name="${prefix}rl_upper_link">
@@ -555,4 +577,5 @@
             <origin rpy="0 0 0" xyz="0.22 0 0"/>
             <limit effort="1000.0" lower="${-134 * deg2rad}" upper="${-7 * deg2rad}" velocity="0.7"/>
+            <dynamics friction="10.0"/>
         </joint>
         <link name="${prefix}rl_under_link">
@@ -579,4 +602,5 @@
             <child link="${prefix}rl_foot"/>
             <origin rpy="0 0 0" xyz="0.22 0 0"/>
+            <dynamics friction="10.0"/>
         </joint>
         <link name="${prefix}rl_foot">
@@ -601,4 +625,5 @@
             <child link="${prefix}rr_hip_roll_actuator"/>
             <origin rpy="0 ${pi/2} 0" xyz="-0.1415 -0.07 0"/>
+            <dynamics friction="10.0"/>
         </joint>
         <link name="${prefix}rr_hip_roll_actuator">
@@ -626,4 +651,5 @@
             <origin rpy="0 0 0" xyz="0 0 0"/>
             <limit effort="1000.0" lower="${-30 * deg2rad}" upper="${30 * deg2rad}" velocity="0.7"/>
+            <dynamics friction="10.0"/>
         </joint>
         <link name="${prefix}rr_hip_pitch_connector">
@@ -651,4 +677,5 @@
             <origin rpy="${pi/2} 0 0" xyz="0 -${rdm_l/2} -0.068"/>
             <limit effort="1000.0" lower="${-51 * deg2rad}" upper="${93 * deg2rad}" velocity="0.7"/>
+            <dynamics friction="10.0"/>
         </joint>
         <link name="${prefix}rr_hip_pitch_actuator">
@@ -674,4 +701,5 @@
             <child link="${prefix}rr_knee_pitch_connector"/>
             <origin rpy="0 0 0" xyz="0 0 0"/>
+            <dynamics friction="10.0"/>
         </joint>
         <link name="${prefix}rr_knee_pitch_connector">
@@ -697,4 +725,5 @@
             <child link="${prefix}rr_knee_pitch_actuator"/>
             <origin rpy="0 0 0" xyz="0 0 0.062"/>
+            <dynamics friction="10.0"/>
         </joint>
         <link name="${prefix}rr_knee_pitch_actuator">
@@ -720,4 +749,5 @@
             <child link="${prefix}rr_upper_link"/>
             <origin rpy="0 0 0" xyz="0 0 0"/>
+            <dynamics friction="10.0"/>
         </joint>
         <link name="${prefix}rr_upper_link">
@@ -746,4 +776,5 @@
             <origin rpy="0 0 0" xyz="0.22 0 0"/>
             <limit effort="1000.0" lower="${-134 * deg2rad}" upper="${-7 * deg2rad}" velocity="0.7"/>
+            <dynamics friction="10.0"/>
         </joint>
         <link name="${prefix}rr_under_link">
@@ -770,4 +801,5 @@
             <child link="${prefix}rr_foot"/>
             <origin rpy="0 0 0" xyz="0.22 0 0"/>
+            <dynamics friction="10.0"/>
         </joint>
         <link name="${prefix}rr_foot">

Commit message: changed damping for leg

File: ros2_ws/src/padwq_description/urdf/padwq.description.xacro (robot description, xacro)
@@ -181,5 +181,5 @@
             <origin rpy="0 0 0" xyz="0.22 0 0"/>
             <limit effort="1000.0" lower="${-134 * deg2rad}" upper="${-7 * deg2rad}" velocity="0.7"/>
-            <dynamics friction="10.0"/>
+            <dynamics damping="1.0" friction="1000.0"/>
         </joint>
         <link name="${prefix}fl_under_link">
@@ -379,5 +379,5 @@
             <origin rpy="0 0 0" xyz="0.22 0 0"/>
             <limit effort="1000.0" lower="${-134 * deg2rad}" upper="${-7 * deg2rad}" velocity="0.7"/>
-            <dynamics friction="10.0"/>
+            <dynamics damping="1.0" friction="1000.0"/>
         </joint>
         <link name="${prefix}fr_under_link">
@@ -577,5 +577,5 @@
             <origin rpy="0 0 0" xyz="0.22 0 0"/>
             <limit effort="1000.0" lower="${-134 * deg2rad}" upper="${-7 * deg2rad}" velocity="0.7"/>
-            <dynamics friction="10.0"/>
+            <dynamics damping="1.0" friction="1000.0"/>
         </joint>
         <link name="${prefix}rl_under_link">
@@ -776,5 +776,5 @@
             <origin rpy="0 0 0" xyz="0.22 0 0"/>
             <limit effort="1000.0" lower="${-134 * deg2rad}" upper="${-7 * deg2rad}" velocity="0.7"/>
-            <dynamics friction="10.0"/>
+            <dynamics damping="1.0" friction="1000.0"/>
         </joint>
         <link name="${prefix}rr_under_link">
