Commit message: updated model; moved mpc demo

File: ros2_ws/src/padwq_description/urdf/padwq.description.xacro (robot description, xacro)
@@ -7,6 +7,7 @@
         <xacro:property name="rdm_r" value="0.049"/>
         <xacro:property name="connector_l" value="0.019"/>
+        <xacro:property name="visual_offset" value="0.001"/>
         <link name="${prefix}base_link">
-            <xacro:inertia_box mass="5.62" x="0.283" y="0.180" z="0.108">
+            <xacro:inertia_box mass="9" x="0.283" y="0.180" z="0.108">
                 <origin xyz="0 0 0" rpy="0 0 0"/>
             </xacro:inertia_box>
@@ -31,5 +32,4 @@
             <child link="${prefix}fl_hip_roll_actuator"/>
             <origin rpy="0 ${pi/2} 0" xyz="0.1415 0.07 0"/>
-            <dynamics friction="10.0"/>
         </joint>
         <link name="${prefix}fl_hip_roll_actuator">
@@ -40,5 +40,5 @@
                 <origin rpy="0 0 0" xyz="0 0 -${rdm_l/2}"/>
                 <geometry>
-                    <cylinder length="${rdm_l}" radius="${rdm_r}"/>
+                    <cylinder length="${rdm_l + visual_offset}" radius="${rdm_r}"/>
                 </geometry>
                 <material name="black"/>
@@ -56,6 +56,6 @@
             <child link="${prefix}fl_hip_pitch_connector"/>
             <origin rpy="0 0 0" xyz="0 0 0"/>
-            <limit effort="1000.0" lower="${-30 * deg2rad}" upper="${30 * deg2rad}" velocity="0.7"/>
-            <dynamics friction="10.0"/>
+            <limit effort="20.0" lower="${-30 * deg2rad}" upper="${30 * deg2rad}" velocity="10"/>
+            <dynamics damping="1.0" friction="1.0"/>
         </joint>
         <link name="${prefix}fl_hip_pitch_connector">
@@ -82,6 +82,6 @@
             <child link="${prefix}fl_hip_pitch_actuator"/>
             <origin rpy="${pi/2} 0 0" xyz="0 ${rdm_l/2} 0.068"/>
-            <limit effort="1000.0" lower="${-51 * deg2rad}" upper="${93 * deg2rad}" velocity="0.7"/>
-            <dynamics friction="10.0"/>
+            <limit effort="20.0" lower="${-51 * deg2rad}" upper="${93 * deg2rad}" velocity="10"/>
+            <dynamics damping="1.0" friction="1.0"/>
         </joint>
         <link name="${prefix}fl_hip_pitch_actuator">
@@ -107,5 +107,4 @@
             <child link="${prefix}fl_knee_pitch_connector"/>
             <origin rpy="0 0 0" xyz="0 0 0"/>
-            <dynamics friction="10.0"/>
         </joint>
         <link name="${prefix}fl_knee_pitch_connector">
@@ -131,5 +130,4 @@
             <child link="${prefix}fl_knee_pitch_actuator"/>
             <origin rpy="0 0 0" xyz="0 0 -0.062"/>
-            <dynamics friction="10.0"/>
         </joint>
         <link name="${prefix}fl_knee_pitch_actuator">
@@ -155,5 +153,4 @@
             <child link="${prefix}fl_upper_link"/>
             <origin rpy="0 0 0" xyz="0 0 0"/>
-            <dynamics friction="10.0"/>
         </joint>
         <link name="${prefix}fl_upper_link">
@@ -180,6 +177,6 @@
             <child link="${prefix}fl_under_link"/>
             <origin rpy="0 0 0" xyz="0.22 0 0"/>
-            <limit effort="1000.0" lower="${-134 * deg2rad}" upper="${-7 * deg2rad}" velocity="0.7"/>
-            <dynamics damping="1.0" friction="1000.0"/>
+            <limit effort="20.0" lower="${7 * deg2rad}" upper="${134 * deg2rad}" velocity="10"/>
+            <dynamics damping="1.0" friction="1.0"/>
         </joint>
         <link name="${prefix}fl_under_link">
@@ -206,5 +203,4 @@
             <child link="${prefix}fl_foot"/>
             <origin rpy="0 0 0" xyz="0.22 0 0"/>
-            <dynamics friction="10.0"/>
         </joint>
         <link name="${prefix}fl_foot">
@@ -229,5 +225,4 @@
             <child link="${prefix}fr_hip_roll_actuator"/>
             <origin rpy="0 ${pi/2} 0" xyz="0.1415 -0.07 0"/>
-            <dynamics friction="10.0"/>
         </joint>
         <link name="${prefix}fr_hip_roll_actuator">
@@ -238,5 +233,5 @@
                 <origin rpy="0 0 0" xyz="0 0 ${-rdm_l/2}"/>
                 <geometry>
-                    <cylinder length="${rdm_l}" radius="${rdm_r}"/>
+                    <cylinder length="${rdm_l + visual_offset}" radius="${rdm_r}"/>
                 </geometry>
                 <material name="black"/>
@@ -254,6 +249,6 @@
             <child link="${prefix}fr_hip_pitch_connector"/>
             <origin rpy="0 0 0" xyz="0 0 0"/>
-            <limit effort="1000.0" lower="${-30 * deg2rad}" upper="${30 * deg2rad}" velocity="0.7"/>
-            <dynamics friction="10.0"/>
+            <limit effort="20.0" lower="${-30 * deg2rad}" upper="${30 * deg2rad}" velocity="10"/>
+            <dynamics damping="1.0" friction="1.0"/>
         </joint>
         <link name="${prefix}fr_hip_pitch_connector">
@@ -280,6 +275,6 @@
             <child link="${prefix}fr_hip_pitch_actuator"/>
             <origin rpy="${pi/2} 0 0" xyz="0 -${rdm_l/2} 0.068"/>
-            <limit effort="1000.0" lower="${-51 * deg2rad}" upper="${93 * deg2rad}" velocity="0.7"/>
-            <dynamics friction="10.0"/>
+            <limit effort="20.0" lower="${-51 * deg2rad}" upper="${93 * deg2rad}" velocity="10"/>
+            <dynamics damping="1.0" friction="1.0"/>
         </joint>
         <link name="${prefix}fr_hip_pitch_actuator">
@@ -305,5 +300,4 @@
             <child link="${prefix}fr_knee_pitch_connector"/>
             <origin rpy="0 0 0" xyz="0 0 0"/>
-            <dynamics friction="10.0"/>
         </joint>
         <link name="${prefix}fr_knee_pitch_connector">
@@ -329,5 +323,4 @@
             <child link="${prefix}fr_knee_pitch_actuator"/>
             <origin rpy="0 0 0" xyz="0 0 0.062"/>
-            <dynamics friction="10.0"/>
         </joint>
         <link name="${prefix}fr_knee_pitch_actuator">
@@ -353,5 +346,4 @@
             <child link="${prefix}fr_upper_link"/>
             <origin rpy="0 0 0" xyz="0 0 0"/>
-            <dynamics friction="10.0"/>
         </joint>
         <link name="${prefix}fr_upper_link">
@@ -378,6 +370,6 @@
             <child link="${prefix}fr_under_link"/>
             <origin rpy="0 0 0" xyz="0.22 0 0"/>
-            <limit effort="1000.0" lower="${-134 * deg2rad}" upper="${-7 * deg2rad}" velocity="0.7"/>
-            <dynamics damping="1.0" friction="1000.0"/>
+            <limit effort="20.0" lower="${7 * deg2rad}" upper="${134 * deg2rad}" velocity="10"/>
+            <dynamics damping="1.0" friction="1.0"/>
         </joint>
         <link name="${prefix}fr_under_link">
@@ -404,5 +396,4 @@
             <child link="${prefix}fr_foot"/>
             <origin rpy="0 0 0" xyz="0.22 0 0"/>
-            <dynamics friction="10.0"/>
         </joint>
         <link name="${prefix}fr_foot">
@@ -427,5 +418,4 @@
             <child link="${prefix}rl_hip_roll_actuator"/>
             <origin rpy="0 ${pi/2} 0" xyz="-0.1415 0.07 0"/>
-            <dynamics friction="10.0"/>
         </joint>
         <link name="${prefix}rl_hip_roll_actuator">
@@ -436,5 +426,5 @@
                 <origin rpy="0 0 0" xyz="0 0 ${rdm_l/2}"/>
                 <geometry>
-                    <cylinder length="${rdm_l}" radius="${rdm_r}"/>
+                    <cylinder length="${rdm_l + visual_offset}" radius="${rdm_r}"/>
                 </geometry>
                 <material name="black"/>
@@ -452,6 +442,6 @@
             <child link="${prefix}rl_hip_pitch_connector"/>
             <origin rpy="0 0 0" xyz="0 0 0"/>
-            <limit effort="1000.0" lower="${-30 * deg2rad}" upper="${30 * deg2rad}" velocity="0.7"/>
-            <dynamics friction="10.0"/>
+            <limit effort="20.0" lower="${-30 * deg2rad}" upper="${30 * deg2rad}" velocity="10"/>
+            <dynamics damping="1.0" friction="1.0"/>
         </joint>
         <link name="${prefix}rl_hip_pitch_connector">
@@ -478,6 +468,6 @@
             <child link="${prefix}rl_hip_pitch_actuator"/>
             <origin rpy="${pi/2} 0 0" xyz="0 ${rdm_l/2} -0.068"/>
-            <limit effort="1000.0" lower="${-51 * deg2rad}" upper="${93 * deg2rad}" velocity="0.7"/>
-            <dynamics friction="10.0"/>
+            <limit effort="20.0" lower="${-51 * deg2rad}" upper="${93 * deg2rad}" velocity="10"/>
+            <dynamics damping="1.0" friction="1.0"/>
         </joint>
         <link name="${prefix}rl_hip_pitch_actuator">
@@ -503,5 +493,4 @@
             <child link="${prefix}rl_knee_pitch_connector"/>
             <origin rpy="0 0 0" xyz="0 0 0"/>
-            <dynamics friction="10.0"/>
         </joint>
         <link name="${prefix}rl_knee_pitch_connector">
@@ -527,5 +516,4 @@
             <child link="${prefix}rl_knee_pitch_actuator"/>
             <origin rpy="0 0 0" xyz="0 0 -0.062"/>
-            <dynamics friction="10.0"/>
         </joint>
         <link name="${prefix}rl_knee_pitch_actuator">
@@ -551,5 +539,4 @@
             <child link="${prefix}rl_upper_link"/>
             <origin rpy="0 0 0" xyz="0 0 0"/>
-            <dynamics friction="10.0"/>
         </joint>
         <link name="${prefix}rl_upper_link">
@@ -576,6 +563,6 @@
             <child link="${prefix}rl_under_link"/>
             <origin rpy="0 0 0" xyz="0.22 0 0"/>
-            <limit effort="1000.0" lower="${-134 * deg2rad}" upper="${-7 * deg2rad}" velocity="0.7"/>
-            <dynamics damping="1.0" friction="1000.0"/>
+            <limit effort="20.0" lower="${7 * deg2rad}" upper="${134 * deg2rad}" velocity="10"/>
+            <dynamics damping="1.0" friction="1.0"/>
         </joint>
         <link name="${prefix}rl_under_link">
@@ -602,5 +589,4 @@
             <child link="${prefix}rl_foot"/>
             <origin rpy="0 0 0" xyz="0.22 0 0"/>
-            <dynamics friction="10.0"/>
         </joint>
         <link name="${prefix}rl_foot">
@@ -625,5 +611,4 @@
             <child link="${prefix}rr_hip_roll_actuator"/>
             <origin rpy="0 ${pi/2} 0" xyz="-0.1415 -0.07 0"/>
-            <dynamics friction="10.0"/>
         </joint>
         <link name="${prefix}rr_hip_roll_actuator">
@@ -634,5 +619,5 @@
                 <origin rpy="0 0 0" xyz="0 0 ${rdm_l/2}"/>
                 <geometry>
-                    <cylinder length="${rdm_l}" radius="${rdm_r}"/>
+                    <cylinder length="${rdm_l + visual_offset}" radius="${rdm_r}"/>
                 </geometry>
                 <material name="black"/>
@@ -650,6 +635,6 @@
             <child link="${prefix}rr_hip_pitch_connector"/>
             <origin rpy="0 0 0" xyz="0 0 0"/>
-            <limit effort="1000.0" lower="${-30 * deg2rad}" upper="${30 * deg2rad}" velocity="0.7"/>
-            <dynamics friction="10.0"/>
+            <limit effort="20.0" lower="${-30 * deg2rad}" upper="${30 * deg2rad}" velocity="10"/>
+            <dynamics damping="1.0" friction="1.0"/>
         </joint>
         <link name="${prefix}rr_hip_pitch_connector">
@@ -676,6 +661,6 @@
             <child link="${prefix}rr_hip_pitch_actuator"/>
             <origin rpy="${pi/2} 0 0" xyz="0 -${rdm_l/2} -0.068"/>
-            <limit effort="1000.0" lower="${-51 * deg2rad}" upper="${93 * deg2rad}" velocity="0.7"/>
-            <dynamics friction="10.0"/>
+            <limit effort="20.0" lower="${-51 * deg2rad}" upper="${93 * deg2rad}" velocity="10"/>
+            <dynamics damping="1.0" friction="1.0"/>
         </joint>
         <link name="${prefix}rr_hip_pitch_actuator">
@@ -701,5 +686,4 @@
             <child link="${prefix}rr_knee_pitch_connector"/>
             <origin rpy="0 0 0" xyz="0 0 0"/>
-            <dynamics friction="10.0"/>
         </joint>
         <link name="${prefix}rr_knee_pitch_connector">
@@ -725,5 +709,4 @@
             <child link="${prefix}rr_knee_pitch_actuator"/>
             <origin rpy="0 0 0" xyz="0 0 0.062"/>
-            <dynamics friction="10.0"/>
         </joint>
         <link name="${prefix}rr_knee_pitch_actuator">
@@ -749,5 +732,4 @@
             <child link="${prefix}rr_upper_link"/>
             <origin rpy="0 0 0" xyz="0 0 0"/>
-            <dynamics friction="10.0"/>
         </joint>
         <link name="${prefix}rr_upper_link">
@@ -759,5 +741,4 @@
                 <geometry>
                     <box size="0.22 0.04 0.04"/>
-                    <!-- <mesh filename="file://$(find padwq_description)/meshes/leg1_5.stl" scale="0.001 0.001 -0.001"/> -->
                 </geometry>
                 <material name="white"/>
@@ -775,6 +756,6 @@
             <child link="${prefix}rr_under_link"/>
             <origin rpy="0 0 0" xyz="0.22 0 0"/>
-            <limit effort="1000.0" lower="${-134 * deg2rad}" upper="${-7 * deg2rad}" velocity="0.7"/>
-            <dynamics damping="1.0" friction="1000.0"/>
+            <limit effort="20.0" lower="${7 * deg2rad}" upper="${134 * deg2rad}" velocity="10"/>
+            <dynamics damping="1.0" friction="1.0"/>
         </joint>
         <link name="${prefix}rr_under_link">
@@ -801,5 +782,4 @@
             <child link="${prefix}rr_foot"/>
             <origin rpy="0 0 0" xyz="0.22 0 0"/>
-            <dynamics friction="10.0"/>
         </joint>
         <link name="${prefix}rr_foot">

File: ros2_ws/src/padwq_description/urdf/padwq.gazebo.xacro (robot description, xacro)
@@ -3,15 +3,10 @@
     <xacro:macro name="gazebo" params="prefix">
         <xacro:macro name="foot_surface">
-            <contact>
-                <min_depth>0.001</min_depth>
-            </contact>
-            <mu1>100.0</mu1>
-            <mu2>100.0</mu2>
-            <kp>1e13</kp>
-            <kd>1.0</kd>
+            <kp>10000000.0</kp>
+            <kd>100000.0</kd>
+            <mu1>10000.0</mu1>
+            <mu2>10000.0</mu2>
+            <maxVel>0.0</maxVel>
             <minDepth>0.001</minDepth>
-            <bounce_threshold>10000000</bounce_threshold>
-            <maxVel>0.1</maxVel>
-            <fdir1>0 0 0</fdir1>
         </xacro:macro>
         <gazebo reference="${prefix}base_link">

File: ros2_ws/src/padwq_description/urdf/padwq.ros2_control.xacro (robot description, xacro)
@@ -17,5 +17,5 @@
                 <command_interface name="position"/>
                 <state_interface name="position">
-                    <param name="initial_value">0.0</param>
+                    <param name="initial_value">${-pi / 4}</param>
                 </state_interface>
                 <state_interface name="velocity"/>
@@ -25,5 +25,5 @@
                 <command_interface name="position"/>
                 <state_interface name="position">
-                    <param name="initial_value">0.0</param>
+                    <param name="initial_value">${pi / 3}</param>
                 </state_interface>
                 <state_interface name="velocity"/>
@@ -41,5 +41,5 @@
                 <command_interface name="position"/>
                 <state_interface name="position">
-                    <param name="initial_value">0.0</param>
+                    <param name="initial_value">${-pi / 4}</param>
                 </state_interface>
                 <state_interface name="velocity"/>
@@ -49,5 +49,5 @@
                 <command_interface name="position"/>
                 <state_interface name="position">
-                    <param name="initial_value">0.0</param>
+                    <param name="initial_value">${pi / 3}</param>
                 </state_interface>
                 <state_interface name="velocity"/>
@@ -65,5 +65,5 @@
                 <command_interface name="position"/>
                 <state_interface name="position">
-                    <param name="initial_value">0.0</param>
+                    <param name="initial_value">${-pi / 4}</param>
                 </state_interface>
                 <state_interface name="velocity"/>
@@ -73,5 +73,5 @@
                 <command_interface name="position"/>
                 <state_interface name="position">
-                    <param name="initial_value">0.0</param>
+                    <param name="initial_value">${pi / 3}</param>
                 </state_interface>
                 <state_interface name="velocity"/>
@@ -89,5 +89,5 @@
                 <command_interface name="position"/>
                 <state_interface name="position">
-                    <param name="initial_value">0.0</param>
+                    <param name="initial_value">${-pi / 4}</param>
                 </state_interface>
                 <state_interface name="velocity"/>
@@ -97,5 +97,5 @@
                 <command_interface name="position"/>
                 <state_interface name="position">
-                    <param name="initial_value">0.0</param>
+                    <param name="initial_value">${pi / 3}</param>
                 </state_interface>
                 <state_interface name="velocity"/>

File: ros2_ws/src/padwq_description/urdf/padwq.urdf.xacro (robot description, xacro)
@@ -6,10 +6,11 @@
     <!-- import robot description -->
     <xacro:include filename="$(find padwq_description)/urdf/padwq.description.xacro"/>
+    <!-- <xacro:include filename="$(find padwq_description)/urdf/padwq_simple.description.xacro"/> -->
     <!-- import gazebo description -->
-    <xacro:include filename="$(find padwq_description)/urdf/gazebo.xacro"/>
+    <xacro:include filename="$(find padwq_description)/urdf/padwq.gazebo.xacro"/>
     <!-- import ros2_control description -->
     <xacro:include filename="$(find padwq_description)/urdf/padwq.ros2_control.xacro"/>
     <xacro:padwq prefix="$(arg prefix)"/>
     <xacro:gazebo prefix="$(arg prefix)"/>
-    <xacro:padwq_ros2_control name="padwq" prefix="$(arg prefix)"/>
+    <xacro:padwq_ros2_control name="GazeboSimSystem" prefix="$(arg prefix)"/>
 </robot>
